Commit message: Fix directional CBF initialization and retryable task aborts, remove the solver timeout and torque limits, and disable Gazebo joint damping. [not tested yet]

File: src/franka_ros/franka_description/robots/common/franka_arm.xacro (robot description, xacro)
@@ -29,5 +29,5 @@
       <axis xyz="0 0 1" />
       <xacro:franka-limits name="joint1" config="${joint_limits}" />
-      <dynamics D="1" K="7000" damping="0.003" friction="0.0" mu_coulomb="0" mu_viscous="16" />
+      <dynamics D="1" K="7000" damping="0.0" friction="0.0" mu_coulomb="0" mu_viscous="16" />
     </joint>
     <xacro:link_with_sc name="link2" gazebo="${gazebo}">
@@ -42,5 +42,5 @@
       <axis xyz="0 0 1" />
       <xacro:franka-limits name="joint2" config="${joint_limits}" />
-      <dynamics D="1" K="7000" damping="0.003" friction="0.0" mu_coulomb="0" mu_viscous="16" />
+      <dynamics D="1" K="7000" damping="0.0" friction="0.0" mu_coulomb="0" mu_viscous="16" />
     </joint>
     <xacro:link_with_sc name="link3" gazebo="${gazebo}">
@@ -55,5 +55,5 @@
       <axis xyz="0 0 1" />
       <xacro:franka-limits name="joint3" config="${joint_limits}" />
-      <dynamics D="1" K="7000" damping="0.003" friction="0.0" mu_coulomb="0" mu_viscous="16" />
+      <dynamics D="1" K="7000" damping="0.0" friction="0.0" mu_coulomb="0" mu_viscous="16" />
     </joint>
     <xacro:link_with_sc name="link4" gazebo="${gazebo}">
@@ -68,5 +68,5 @@
       <axis xyz="0 0 1" />
       <xacro:franka-limits name="joint4" config="${joint_limits}" />
-      <dynamics D="1" K="7000" damping="0.003" friction="0.0" mu_coulomb="0" mu_viscous="16" />
+      <dynamics D="1" K="7000" damping="0.0" friction="0.0" mu_coulomb="0" mu_viscous="16" />
     </joint>
     <xacro:link_with_sc name="link5" gazebo="${gazebo}">
@@ -82,5 +82,5 @@
       <axis xyz="0 0 1" />
       <xacro:franka-limits name="joint5" config="${joint_limits}" />
-      <dynamics D="1" K="7000" damping="0.003" friction="0.0" mu_coulomb="0" mu_viscous="16" />
+      <dynamics D="1" K="7000" damping="0.0" friction="0.0" mu_coulomb="0" mu_viscous="16" />
     </joint>
     <xacro:link_with_sc name="link6" gazebo="${gazebo}">
@@ -95,5 +95,5 @@
       <axis xyz="0 0 1" />
       <xacro:franka-limits name="joint6" config="${joint_limits}" />
-      <dynamics D="1" K="7000" damping="0.003" friction="0.0" mu_coulomb="0" mu_viscous="16" />
+      <dynamics D="1" K="7000" damping="0.0" friction="0.0" mu_coulomb="0" mu_viscous="16" />
     </joint>
     <xacro:link_with_sc name="link7" gazebo="${gazebo}" rpy="0 0 ${pi/4}">
@@ -109,5 +109,5 @@
       <axis xyz="0 0 1"/>
       <xacro:franka-limits name="joint7" config="${joint_limits}" />
-      <dynamics D="1" K="7000" damping="0.003" friction="0.0" mu_coulomb="0" mu_viscous="16"/>
+      <dynamics D="1" K="7000" damping="0.0" friction="0.0" mu_coulomb="0" mu_viscous="16"/>
     </joint>
     <link name="${arm_id}_link8"/>
